File: hardware/IMU.sch (KiCad schematic (older format))
At the start: 8 parts, among them J6 Conn_01x08, U4 MPU-6050

Commit message: PCB layout
Parts:
- removed J6: Conn_01x08, Board:MPU6050_Breakout, symbol Connector_Generic:Conn_01x08
- added J6: Conn_01x04, Board:Wire-Pad-01x04, symbol Connector_Generic:Conn_01x04
- renumbered R14 to R10, R15 to R11, R16 to R12, R13 to R9
Connections:
- net +3V3: now also J6.4 (Pin_4)
- net GND: now also J6.3 (Pin_3)
- net SCL: now also J6.2 (Pin_2)
- net SDA: now also J6.1 (Pin_1)
- net AD0: no longer names the net of R10.1, U4.9 (AD0)
- net INT: no longer names the net of R12.2, U4.12 (INT)
- net XCL: no longer names the net of U4.7 (AUX_SCL)
- net XDA: no longer names the net of U4.6 (AUX_SDA)
- no-connect marks 0 -> 2
Changed lines of the file:
@@
 P 4800 2975
 AR Path="/6233C83C/623F7798" Ref="R?"  Part="1"
-AR Path="/623EC3BB/623F7798" Ref="R13"  Part="1"
-F 0 "R13" H 4868 3021 50  0000 L CNN
+AR Path="/623EC3BB/623F7798" Ref="R9"  Part="1"
+F 0 "R9" H 4868 3021 50  0000 L CNN
 F 1 "10k" H 4868 2930 50  0000 L CNN
 F 2 "Resistor_SMD:R_0805_2012Metric_Pad1.20x1.40mm_HandSolder" H 4800 2975 50  0001 C CNN
@@
 P 5100 2975
 AR Path="/6233C83C/623F779E" Ref="R?"  Part="1"
-AR Path="/623EC3BB/623F779E" Ref="R15"  Part="1"
-F 0 "R15" H 5168 3021 50  0000 L CNN
+AR Path="/623EC3BB/623F779E" Ref="R11"  Part="1"
+F 0 "R11" H 5168 3021 50  0000 L CNN
 F 1 "10k" H 5168 2930 50  0000 L CNN
 F 2 "Resistor_SMD:R_0805_2012Metric_Pad1.20x1.40mm_HandSolder" H 5100 2975 50  0001 C CNN
@@
 P 6000 4575
 AR Path="/6233C83C/623F77B3" Ref="#PWR?"  Part="1"
-AR Path="/623EC3BB/623F77B3" Ref="#PWR038"  Part="1"
-F 0 "#PWR038" H 6000 4325 50  0001 C CNN
+AR Path="/623EC3BB/623F77B3" Ref="#PWR035"  Part="1"
+F 0 "#PWR035" H 6000 4325 50  0001 C CNN
 F 1 "GND" H 6005 4402 50  0000 C CNN
 F 2 "" H 6000 4575 50  0001 C CNN
@@
 P 4850 3925
 AR Path="/6233C83C/623F77D6" Ref="#PWR?"  Part="1"
-AR Path="/623EC3BB/623F77D6" Ref="#PWR034"  Part="1"
-F 0 "#PWR034" H 4850 3675 50  0001 C CNN
+AR Path="/623EC3BB/623F77D6" Ref="#PWR031"  Part="1"
+F 0 "#PWR031" H 4850 3675 50  0001 C CNN
 F 1 "GND" H 4855 3752 50  0000 C CNN
 F 2 "" H 4850 3925 50  0001 C CNN
@@
 P 7200 4375
 AR Path="/6233C83C/623F77DC" Ref="#PWR?"  Part="1"
-AR Path="/623EC3BB/623F77DC" Ref="#PWR040"  Part="1"
-F 0 "#PWR040" H 7200 4125 50  0001 C CNN
+AR Path="/623EC3BB/623F77DC" Ref="#PWR037"  Part="1"
+F 0 "#PWR037" H 7200 4125 50  0001 C CNN
 F 1 "GND" H 7205 4202 50  0000 C CNN
 F 2 "" H 7200 4375 50  0001 C CNN
@@
 	1    0    0    -1
 $EndComp
-Text Label 7350 3275 2    50   ~ 0
-INT
 $Comp
 L power:+3.3V #PWR?
@@
 P 4950 2675
 AR Path="/6233C83C/623F77E3" Ref="#PWR?"  Part="1"
-AR Path="/623EC3BB/623F77E3" Ref="#PWR035"  Part="1"
-F 0 "#PWR035" H 4950 2525 50  0001 C CNN
+AR Path="/623EC3BB/623F77E3" Ref="#PWR032"  Part="1"
+F 0 "#PWR032" H 4950 2525 50  0001 C CNN
 F 1 "+3.3V" H 4965 2848 50  0000 C CNN
 F 2 "" H 4950 2675 50  0001 C CNN
@@
 	4950 2825 5100 2825
 Wire Wire Line
-	6700 3475 6950 3475
-Wire Wire Line
-	6700 3575 6950 3575
-Text Label 6950 3475 2    50   ~ 0
-XDA
-Text Label 6950 3575 2    50   ~ 0
-XCL
-Wire Wire Line
-	4550 3475 4850 3475
-Wire Wire Line
 	4850 3475 4850 3625
-Connection ~ 4850 3475
 $Comp
 L Device:R_Small_US R?
@@
 P 4850 3725
 AR Path="/6233C83C/623F77FD" Ref="R?"  Part="1"
-AR Path="/623EC3BB/623F77FD" Ref="R14"  Part="1"
-F 0 "R14" H 4918 3771 50  0000 L CNN
+AR Path="/623EC3BB/623F77FD" Ref="R10"  Part="1"
+F 0 "R10" H 4918 3771 50  0000 L CNN
 F 1 "4.7k" H 4918 3680 50  0000 L CNN
 F 2 "Resistor_SMD:R_0805_2012Metric_Pad1.20x1.40mm_HandSolder" H 4850 3725 50  0001 C CNN
@@
 	1    0    0    -1
 $EndComp
-Text Label 4550 3475 0    50   ~ 0
-AD0
 $Comp
 L Device:R_Small_US R?
@@
 P 6950 3075
 AR Path="/6233C83C/623F7804" Ref="R?"  Part="1"
-AR Path="/623EC3BB/623F7804" Ref="R16"  Part="1"
-F 0 "R16" H 7018 3121 50  0000 L CNN
+AR Path="/623EC3BB/623F7804" Ref="R12"  Part="1"
+F 0 "R12" H 7018 3121 50  0000 L CNN
 F 1 "10k" H 7018 3030 50  0000 L CNN
 F 2 "Resistor_SMD:R_0805_2012Metric_Pad1.20x1.40mm_HandSolder" H 6950 3075 50  0001 C CNN
@@
 P 6950 2875
 AR Path="/6233C83C/623F780A" Ref="#PWR?"  Part="1"
-AR Path="/623EC3BB/623F780A" Ref="#PWR039"  Part="1"
-F 0 "#PWR039" H 6950 2725 50  0001 C CNN
+AR Path="/623EC3BB/623F780A" Ref="#PWR036"  Part="1"
+F 0 "#PWR036" H 6950 2725 50  0001 C CNN
 F 1 "+3.3V" H 6965 3048 50  0000 C CNN
 F 2 "" H 6950 2875 50  0001 C CNN
@@
 Wire Wire Line
 	6950 3175 6950 3275
-Connection ~ 6950 3275
-Wire Wire Line
-	6950 3275 7350 3275
 Wire Wire Line
 	6950 2875 6950 2975
@@
 P 5150 4075
 AR Path="/6233C83C/623F7815" Ref="#PWR?"  Part="1"
-AR Path="/623EC3BB/623F7815" Ref="#PWR036"  Part="1"
-F 0 "#PWR036" H 5150 3825 50  0001 C CNN
+AR Path="/623EC3BB/623F7815" Ref="#PWR033"  Part="1"
+F 0 "#PWR033" H 5150 3825 50  0001 C CNN
 F 1 "GND" H 5155 3902 50  0000 C CNN
 F 2 "" H 5150 4075 50  0001 C CNN
@@
 P 6000 2625
 AR Path="/6233C83C/623F783D" Ref="#PWR?"  Part="1"
-AR Path="/623EC3BB/623F783D" Ref="#PWR037"  Part="1"
-F 0 "#PWR037" H 6000 2475 50  0001 C CNN
+AR Path="/623EC3BB/623F783D" Ref="#PWR034"  Part="1"
+F 0 "#PWR034" H 6000 2475 50  0001 C CNN
 F 1 "+3.3V" H 6015 2798 50  0000 C CNN
 F 2 "" H 6000 2625 50  0001 C CNN
@@
 $EndComp
 $Comp
-L Connector_Generic:Conn_01x08 J6
-U 1 1 624929F5
-P 3100 3600
-F 0 "J6" H 3018 2975 50  0000 C CNN
-F 1 "Conn_01x08" H 3018 3066 50  0000 C CNN
-F 2 "Board:MPU6050_Breakout" H 3100 3600 50  0001 C CNN
-F 3 "~" H 3100 3600 50  0001 C CNN
-	1    3100 3600
-	-1   0    0    1
-$EndComp
-$Comp
 L power:+3.3V #PWR?
 U 1 1 624969A6
 P 3750 3150
 AR Path="/6233C83C/624969A6" Ref="#PWR?"  Part="1"
-AR Path="/623EC3BB/624969A6" Ref="#PWR032"  Part="1"
-F 0 "#PWR032" H 3750 3000 50  0001 C CNN
+AR Path="/623EC3BB/624969A6" Ref="#PWR029"  Part="1"
+F 0 "#PWR029" H 3750 3000 50  0001 C CNN
 F 1 "+3.3V" H 3765 3323 50  0000 C CNN
 F 2 "" H 3750 3150 50  0001 C CNN
@@
 P 3750 3350
 AR Path="/6233C83C/6249A79C" Ref="#PWR?"  Part="1"
-AR Path="/623EC3BB/6249A79C" Ref="#PWR033"  Part="1"
-F 0 "#PWR033" H 3750 3100 50  0001 C CNN
+AR Path="/623EC3BB/6249A79C" Ref="#PWR030"  Part="1"
+F 0 "#PWR030" H 3750 3100 50  0001 C CNN
 F 1 "GND" H 3755 3177 50  0000 C CNN
 F 2 "" H 3750 3350 50  0001 C CNN
@@
 Text Label 3600 3500 2    50   ~ 0
 SDA
-Wire Wire Line
-	3300 3600 3600 3600
-Text Label 3600 3600 2    50   ~ 0
-XDA
-Wire Wire Line
-	3300 3700 3600 3700
-Text Label 3600 3700 2    50   ~ 0
-XCL
-Wire Wire Line
-	3300 3800 3600 3800
-Text Label 3600 3800 2    50   ~ 0
-AD0
-Wire Wire Line
-	3300 3900 3600 3900
-Text Label 3600 3900 2    50   ~ 0
-INT
+$Comp
+L Connector_Generic:Conn_01x04 J6
+U 1 1 6241E801
+P 3100 3400
+F 0 "J6" H 3018 2975 50  0000 C CNN
+F 1 "Conn_01x04" H 3018 3066 50  0000 C CNN
+F 2 "Board:Wire-Pad-01x04" H 3100 3400 50  0001 C CNN
+F 3 "~" H 3100 3400 50  0001 C CNN
+	1    3100 3400
+	-1   0    0    1
+$EndComp
+NoConn ~ 6700 3475
+NoConn ~ 6700 3575
 $EndSCHEMATC
