File: hardware/BMS.sch (KiCad schematic (older format))
At the start: 28 parts, among them IC1 DW01A, P1 USB_C_Plug_USB2.0, Q3 AO3401A, Q4 FS8205A, SW3 SW_SPST, U5 MT3608, U6 TP4056

Commit message: PCB layout
Parts:
- removed BATT+1, BATT-1: TestPoint, Board:Wire-Pad, symbol Connector:TestPoint
- removed C8: 10uF, Capacitor_SMD:C_0805_2012Metric_Pad1.18x1.45mm_HandSolder, symbol Device:CP_Small
- added J7: Conn_01x02, Board:Wire-Pad-01x02, symbol Connector_Generic:Conn_01x02
- renumbered D8 to D6, D9 to D7, D10 to D8, D11 to D9, R17 to R13, R18 to R14, R19 to R15, R20 to R16, R21 to R17, R22 to R18, R23 to R19, R24 to R20, R25 to R21, R26 to R22
Connections:
- net BATT+: now also J7.1 (Pin_1)
- net BATT-: now also J7.2 (Pin_2)
Other:
- moved on the sheet: R20, R21

Commit message: PCB routed
Parts:
- SW3: footprint Button_Switch_SMD:SW_SPDT_PCM12 -> Board:SW_SPDT_PCM12
Changed lines of the file:
@@
 F 0 "SW3" H 2075 6085 50  0000 C CNN
 F 1 "SW_SPST" H 2075 5994 50  0000 C CNN
-F 2 "Button_Switch_SMD:SW_SPDT_PCM12" H 2075 5850 50  0001 C CNN
+F 2 "Board:SW_SPDT_PCM12" H 2075 5850 50  0001 C CNN
 F 3 "~" H 2075 5850 50  0001 C CNN
 	1    2075 5850
