File: hardware/board.kicad_pcb (KiCad board)
At the start: 2 copper layers, 150 x 40 mm, 79 parts, among them IC1 DW01A, J1 Conn_01x03_Male, J2 Conn_01x03_Male, J3 Conn_01x06, J4 Conn_01x06_Female, J5 Conn_01x06, J6 Conn_01x04, J7 Conn_01x02, J8 Conn_01x04, P1 USB_C_Plug_USB2.0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

Commit message: PCB: Minor changes
Parts:
- moved H2 23.6 mm to (187.2, 97.5)
- moved C1 23.4 mm to (155.2, 108.2)
- moved C2 23.4 mm to (149.2, 108.2)
- moved C3 23.4 mm to (150.1, 93.5)
- moved C4 23.4 mm to (151.9, 97.5)
- moved C5 23.4 mm to (136.1, 91.6)
- moved C6 23.4 mm to (138.8, 91.6)
- moved C7 23.4 mm to (158.8, 108.1)
- moved D1 23.4 mm to (103.2, 97.5)
- moved D10 23.4 mm to (160.0, 103.2)
- moved D2 23.4 mm to (147.8, 117.9)
- moved D3 23.4 mm to (95.8, 100.5)
- moved D4 23.4 mm to (199.8, 100.5)
- moved D5 23.4 mm to (192.2, 97.5)
- moved D6 23.4 mm to (156.0, 116.3)
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