File: hardware/board.sch (KiCad schematic (older format))
At the start: 41 parts, among them J1 Conn_01x03_Male, J2 Conn_01x03_Male, J3 Conn_01x06, J4 Conn_01x06_Female, J5 Conn_01x06, J8 Conn_01x04, Q1 AO3400A, Q2 AO3400A, SW1 SW_Push, SW2 SW_Push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

Commit message: PCB: Minor changes
Other:
- moved on the sheet: C1, C2, D1, D10, D2, D3, D4, D5, H1, H2, H3, H4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
